File: kicad/water-sensor.kicad_pcb (KiCad board)
At the start: 2 copper layers, 7 parts, among them U1 ATMEGA8-16AU

Commit message: End work 1803
Parts:
- added CON1: AVR-ISP6, w_pin_strip:pin_strip_3x2, F.Cu at (109.2, 67.3)
- added Q1: BC847, TO_SOT_Packages_SMD:SOT-23, F.Cu at (116.4, 60.5)
- added R4: 10k, Resistors_SMD:R_0805, F.Cu at (120.9, 59.7)
- added U2: LM78L05ACZ, TO_SOT_Packages_THT:TO-92_Molded_Narrow, F.Cu at (108.0, 57.1)
- C1: value 100n -> 0,47
- R1: value 100 -> 10k
- U1: value ATMEGA8-16AU -> ATTINY13A-SSU; footprint Housings_QFP:TQFP-32_7x7mm_Pitch0.8mm -> Housings_SOIC:SOIC-8_3.9x4.9mm_Pitch1.27mm
Connections:
- C1 pad 1: GND -> Net-(C1-Pad1)
- C1 pad 2: Net-(C1-Pad2) -> GND
- R1 pad 1: +5V -> Net-(C1-Pad1)
- R1 pad 2: Net-(C1-Pad2) -> Net-(R1-Pad2)
- R2 pad 2: Net-(R2-Pad2) -> Net-(C1-Pad1)
- R3 pad 2: Net-(R2-Pad2) -> Net-(C1-Pad1)
- U1 pad 3: GND -> Net-(R1-Pad2)
- U1 pad 4: +5V -> GND
- U1 pad 5: GND -> Net-(CON1-Pad4)
- U1 pad 6: +5V -> Net-(CON1-Pad1)
- U1 pad 8: Net-(U1-Pad8) -> +5V
