File: kicad/water-sensor.sch (KiCad schematic (older format))
At the start: 1 part, among them U1 ATMEGA8-16AU

Commit message: End work_13.03
Parts:
- added C1, C2, C3: 100n, Capacitors_SMD:C_0805, symbol C
- added R1: 100, Resistors_SMD:R_0805, symbol R
- added R2, R3: 510k, Resistors_SMD:R_0805, symbol R
Connections:
- net at U1.20 (AREF): now also C1.2, R1.2
- net GND: now reaches U1.21 (AGND)
- net GND: now also U1.3 (GND), U1.5 (GND), C1.1, C2.2, C3.2, R3.1
- net at U1.23 ((ADC0)PC0): now also R2.2, R3.2
- net +5V: now reaches U1.4 (VCC)
- net +5V: now also U1.6 (VCC), C2.1, C3.1, R1.1, R2.1

Commit message: End work 1803
Parts:
- removed C1: 100n, Capacitors_SMD:C_0805, symbol C
- removed R1: 100, Resistors_SMD:R_0805, symbol R
- removed U1: ATMEGA8-16AU, Housings_QFP:TQFP-32_7x7mm_Pitch0.8mm, symbol ATMEGA8-16AU
- added C1: 0,47, Capacitors_SMD:C_0805, symbol C-RESCUE-water-sensor
- added CON1: AVR-ISP6, w_pin_strip:pin_strip_3x2, symbol AVR-ISP6
- added D1: D_Schottky_x2_Serial_AKC, symbol D_Schottky_x2_Serial_AKC
- added Q1: BC847, TO_SOT_Packages_SMD:SOT-23, symbol BC847
- added R1, R4: 10k, Resistors_SMD:R_0805, symbol R-RESCUE-water-sensor
- added U1: ATTINY13A-SSU, Housings_SOIC:SOIC-8_3.9x4.9mm_Pitch1.27mm, symbol ATTINY13A-SSU
- added U2: LM78L05ACZ, TO_SOT_Packages_THT:TO-92_Molded_Narrow, symbol LM78L05ACZ
- C2, C3: symbol C -> C-RESCUE-water-sensor
- R2, R3: symbol R -> R-RESCUE-water-sensor
Connections:
- net +5V: now also CON1.2 (Vcc), D1.2 (K), U1.8 (VCC), U2.1 (OUT)
- net GND: now also C1.2, CON1.6 (GND), D1.1 (A), Q1.2 (E), U1.4 (GND), U2.2 (GND)
- net at R2.2, R3.2: now also C1.1, D1.3 (common), R1.1
- new net: CON1.1 (MISO), U1.6 (PB1(MISO/AIN1/OC0B/INT0/PCINT1))
- new net: CON1.3 (SCK), U1.7 (PB2(SCK/ADC1/T0/PCINT2))
- new net: CON1.4 (MOSI), U1.5 (PB0(MOSI/AIN0/OC0A/PCINT0))
- new net: CON1.5 (RST), U1.1 (PB5(~RESET~/ADC0/PCINT5/dW))
- new net: R1.2, U1.3 (PB4(ADC2/PCINT4))
- new net: R4.1, U1.2 (PB3(CLKI/ADC3/PCINT3))
- new net: Q1.1 (B), R4.2
Other:
- moved on the sheet: R2, R3
